File: bsides_badge.sch (KiCad schematic (older format))
At the start: 5 parts, among them J1 Conn_01x16, J2 Conn_01x01

Commit message: Change to credit card format and rebalanced battery
Parts:
- J1: footprint Pin_Headers:Pin_Header_Straight_1x16_Pitch2.54mm -> TestPoint:TestPoint_Pad_1.0x1.0mm
- J2: footprint Pin_Headers:Pin_Header_Straight_1x01_Pitch2.54mm -> TestPoint:TestPoint_Pad_2.0x2.0mm
Changed lines of the file:
@@
 F 0 "J1" H 1350 2650 50  0000 C CNN
 F 1 "Conn_01x16" H 1350 950 50  0000 C CNN
-F 2 "Pin_Headers:Pin_Header_Straight_1x16_Pitch2.54mm" H 1350 1850 50  0001 C CNN
+F 2 "TestPoint:TestPoint_Pad_1.0x1.0mm" H 1350 1850 50  0001 C CNN
 F 3 "" H 1350 1850 50  0001 C CNN
 	1    1350 1850
@@
 F 0 "J2" H 2450 2850 50  0000 C CNN
 F 1 "Conn_01x01" H 2450 2650 50  0000 C CNN
-F 2 "Pin_Headers:Pin_Header_Straight_1x01_Pitch2.54mm" H 2450 2750 50  0001 C CNN
+F 2 "TestPoint:TestPoint_Pad_2.0x2.0mm" H 2450 2750 50  0001 C CNN
 F 3 "" H 2450 2750 50  0001 C CNN
 	1    2450 2750
